Commit message: amigobot: add webcam frame, reformat

File: src/amigobot/urdf/amigobot.urdf.xacro (robot description, xacro)
@@ -8,5 +8,5 @@
   <!--<include filename="$(find amr_robots_description)/urdf/materials.xacro"/>-->
   <xacro:include filename="$(find amr_robots_description)/urdf/pioneer3dx_wheel.xacro"/>
-<!-- Chassis -->
+    <!-- Chassis -->
 	<link name="base_link">
 		<inertial>
@@ -35,244 +35,285 @@
 		</collision>
 	</link>
-	<link name="sonar">
-		<inertial>
-			<mass value="0.0001"/>
-			<origin xyz="0 0 0"/>
-			<inertia ixx="1" ixy="0" ixz="0"
-				 iyy="1" iyz="0" izz="1"/>
-		</inertial>
-		<visual name="pioneer_geom">
-			<origin xyz="0 0 0" rpy="0 0 0"/>
-			<geometry name="pioneer_geom">
-				<mesh filename="package://amr_robots_description/meshes/p3dx_meshes/front_sonar.stl"/>
-			</geometry>
-			<material name="SonarYellow">
-				<color rgba="0.715 0.583 0.210 1.0"/>
-			</material>
-		</visual>
-		<collision>
-			<origin xyz="0 0 0" rpy="0 0 0"/>
-			<geometry>
-				<box size="0 0 0"/>
-			</geometry>
-		</collision>
-	</link>
-	<gazebo reference="sonar">
-		<material value="Gazebo/Yellow"/>
-	</gazebo>
-	<joint name="base_front_joint" type="fixed">
-		<origin xyz="-0.198 0 0.208" rpy="0 0 0"/>
-		<parent link="base_link"/>
-		<child link="sonar"/>
-	</joint>
-	<!-- Caster -->
-	<joint name="base_caster_swivel_joint" type="continuous">
-		<origin xyz="-0.185 0 0.055" rpy="0 0 0"/>
-		<anchor xyz="0 0 0"/>
-    	<limit effort="100" velocity="100" k_velocity="0" />
-    	<joint_properties damping="0.0" friction="0.0" />
-		<parent link="base_link"/>
-		<child link="caster_swivel"/>
-	</joint>
-	<link name="caster_swivel">
-		<inertial>
-			<mass value="0.1"/>
-			<origin xyz="0 0 0"/>
-			<inertia ixx="0.01" ixy="0" ixz="0"
-				 iyy="0.01" iyz="0" izz="0.01"/>
-  	 	</inertial>
-	<visual name="pioneer_geom">
-		<origin xyz="0 0 0" rpy="0 0 0"/>
-		<geometry name="pioneer_geom">
-			<mesh filename="package://amr_robots_description/meshes/p3dx_meshes/caster_swivel.stl"/>
-		</geometry>
-		<material name="caster_swivel">
-			<color rgba="0.5 0.5 0.5 1"/>
-		</material>
-	</visual>
-	<collision>
-		<origin xyz="0 0 0" rpy="0 0 0"/>
-		<geometry>
-			<box size="0 0 0"/>
-		</geometry>
-	</collision>
-	</link>
-	<gazebo reference="caster_swivel">
-		<material value="Gazebo/Grey"/>
-	</gazebo>
-<!-- Center Wheel + Hubcap -->
-	<link name="caster_hubcap">
-		<inertial>
-			<mass value="0.01"/>
-			<origin xyz="0 0 0"/>
-			<inertia ixx="0.012411765597" ixy="-0.000711733678" ixz="0.00050272983"
-				 iyy="0.015218160428" iyz="-0.000004273467" izz="0.011763977943"/>
-  	 	</inertial>
-	<visual name="pioneer_geom">
-		<origin xyz="0 0 0" rpy="0 0 0"/>
-		<geometry name="pioneer_geom">
-			<mesh filename="package://amr_robots_description/meshes/p3dx_meshes/caster_hubcap.stl"/>
-		</geometry>
-		<material name="caster_swivel">
-			<color rgba="0.5 0.5 0.5 1"/>
-		</material>
-	</visual>
-	<collision>
-		<origin xyz="0 0 0" rpy="0 0 0"/>
-		<geometry>
-			<box size="0.05 0.05 0.05"/>
-		</geometry>
-	</collision>
-	</link>
-	<gazebo reference="caster_hubcap">
-		<material value="Gazebo/Grey"/>
-	</gazebo>
-	<joint name="caster_swivel_hubcap_joint" type="continuous">
-		<origin xyz="-0.026 0 -0.016" rpy="0 0 0"/>
-		<axis xyz="0 1 0"/>
-		<anchor xyz="0 0 0"/>
-    <limit effort="100" velocity="100" k_velocity="0" />
-    <joint_properties damping="0.0" friction="0.0" />
-	  <parent link="caster_swivel"/>
-		<child link="caster_wheel"/>
-	</joint>
-	<link name="caster_wheel">
-		<inertial>
-			<mass value="0.1"/>
-			<origin xyz="0 0 0"/>
-			<inertia ixx="0.012411765597" ixy="-0.000711733678" ixz="0.00050272983"
-				 iyy="0.015218160428" iyz="-0.000004273467" izz="0.011763977943"/>
-  	 	</inertial>
-	<visual name="pioneer_geom">
-		<origin xyz="0 0 0" rpy="0 0 0"/>
-		<geometry name="pioneer_geom">
-			<mesh filename="package://amr_robots_description/meshes/p3dx_meshes/caster_wheel.stl"/>
-		</geometry>
-		<material name="WheelBlack">
-			<color rgba="0.117 0.117 0.117 1"/>
-		</material>
-	</visual>
-	<collision>
-		<origin xyz="0 0 0" rpy="${-3.1415927/2.0} 0 0"/>
-		<geometry>
-			<!--<mesh filename="package://amr_robots_description/meshes/p3dx_meshes/caster_wheel.stl"/>-->
-			<cylinder radius="0.0375" length="0.01"/>
-		</geometry>
-	</collision>
-	</link>
-	<gazebo reference="left_hub">
-		<material value="Gazebo/Yellow"/>
-	</gazebo>
-	<joint name="caster_wheel_joint" type="fixed">
-		<origin xyz="-0.0035 0 -0.001" rpy="0 0 0"/>
-		<parent link="caster_wheel"/>
-		<child link="caster_hubcap"/>
-	</joint>
-	<link name="left_hub">
-		<visual>
-			<origin xyz="0 0 0" rpy="0 0 0"/>
-			<geometry>
-				<mesh filename="package://amr_robots_description/meshes/p3dx_meshes/left_hubcap.stl"/>
-			</geometry>
-			<material name="HubcapYellow">
-				<color rgba="1.0 0.811 0.151 1.0"/>
-			</material>
-		</visual>
-		<collision>
-			<origin xyz="0 0 0" rpy="${-3.1415927/2.0} 0 0"/>
-			<geometry>
-				<!--<mesh filename="package://amr_robots_description/meshes/p3dx_meshes/caster_wheel.stl"/>-->
-				<cylinder radius="0.09" length="0.01"/>
-			</geometry>
-		</collision>
-	</link>
-	<joint name="left_hub_joint" type="fixed">
-		<origin xyz="0 0.15 0.08" rpy="0 0 0"/>
-		<parent link="base_link"/>
-		<child link="left_hub"/>
-		<axis xyz="0 1 0"/>
-	</joint>
-	<link name="left_wheel">
-		<visual>
-			<origin xyz="0 0 0" rpy="0 0 0"/>
-			<geometry>
-				<mesh filename="package://amr_robots_description/meshes/p3dx_meshes/left_wheel.stl"/>
-			</geometry>
-			<material name="WheelBlack">
-				<color rgba="0.117 0.117 0.117 1"/>
-			</material>
-		</visual>
-	</link>
-	<joint name="left_wheel_joint" type="fixed"> <!-- type="continuous" -->
-		<origin xyz="0 0 0" rpy="0 0 0"/>
-		<parent link="left_hub"/>
-		<child link="left_wheel"/>
-	</joint>
-	<gazebo reference="left_wheel_joint">
-		<material value="Gazebo/Black"/>
-	</gazebo>
-	<link name="right_hub">
-		<visual>
-			<origin xyz="0 0 0" rpy="0 0 0"/>
-			<geometry>
-				<mesh filename="package://amr_robots_description/meshes/p3dx_meshes/right_hubcap.stl"/>
-			</geometry>
-			<material name="HubcapYellow">
-				<color rgba="1.0 0.811 0.151 1.0"/>
-			</material>
-		</visual>
-		<collision>
-		<origin xyz="0 0 0" rpy="${-3.1415927/2.0} 0 0"/>
-		<geometry>
-			<!--<mesh filename="package://amr_robots_description/meshes/p3dx_meshes/caster_wheel.stl"/>-->
-			<cylinder radius="0.09" length="0.01"/>
-		</geometry>
-	</collision>
-	</link>
-	<gazebo reference="right_hub">
-		<material value="Gazebo/Yellow"/>
-	</gazebo>
-	<joint name="right_hub_joint" type="fixed">
-		<origin xyz="0 -0.15 0.08" rpy="0 0 0"/>
-		<parent link="base_link"/>
-		<child link="right_hub"/>
-		<axis xyz="0 1 0"/>
-	</joint>
-	<link name="right_wheel">
-		<visual>
-			<origin xyz="0 0 0" rpy="0 0 0"/>
-			<geometry>
-				<mesh filename="package://amr_robots_description/meshes/p3dx_meshes/right_wheel.stl"/>
-			</geometry>
-			<material name="WheelBlack">
-				<color rgba="0.117 0.117 0.117 1"/>
-			</material>
-		</visual>
-	</link>
-	<joint name="right_wheel_joint" type="fixed"> <!-- type="continuous" -->
-		<origin xyz="0 0 0" rpy="0 0 0"/>
-		<parent link="right_hub"/>
-		<child link="right_wheel"/>
-	</joint>
-	<gazebo reference="right_wheel_joint">
-		<material value="Gazebo/Black"/>
-	</gazebo>
-<gazebo>
-	<plugin name="differential_drive_controller" filename="libgazebo_ros_diff_drive.so">
-    <alwaysOn>true</alwaysOn>
-		<updateRate>100</updateRate>
-		<leftJoint>left_wheel_joint</leftJoint>
-		<rightJoint>right_wheel_joint</rightJoint>
-		<wheelSeparation>0.158</wheelSeparation>
-		<wheelDiameter>0.10</wheelDiameter>
-		<torque>5</torque>
-		<!-- interface:position name="position_iface_0"/ -->
-    <commandTopic>cmd_vel</commandTopic>
-    <robotBaseFrame>base_link</robotBaseFrame>
-    <odometryTopic>odom</odometryTopic>
-    <odometryFrame>odom</odometryFrame>
-	</plugin>
-  <!-- TODO include P3D (ground truth) plugin -->
-  <!-- XXX old urdf included a gazebo_ros_controller_manager plugin with a 1 second update rate -->
-</gazebo>
+    <!-- Camera; mounted on top front of robot; rotated to the right.
+         load the xacro with
+         <param name="robot_description" command="$(find xacro)/xacro.py $(arg model) use_web_cam:=false" />
+         to not add a camera.
+         For a camera, the z axis is in the direction of the view, x goes to
+         the right (wrt/ view direction) and y downwards.
+         -->
+    <xacro:arg name="use_web_cam" default="true"/>
+    <xacro:if value="$(arg use_web_cam)">
+        <link name="web_cam">
+            <inertial>
+                <mass value="0.05" />
+                <origin xyz="0 0 0" rpy="0 0 0"/>
+                <inertia ixx="1e-6" ixy="0" ixz="0" iyy="1e-6" iyz="0" izz="1e-6" />
+            </inertial>
+            <collision>
+                <origin xyz="0 0 0" rpy="0 0 0"/>
+                <geometry>
+                    <box size="0.2 0.12 0.2" /> <!-- larger box to include stand -->
+                </geometry>
+            </collision>
+            <visual>
+                <origin xyz="0 0 0" rpy="0 0 0"/>
+                <geometry>
+                    <box size="0.07 0.1 0.025"/>
+                </geometry>
+                <material name="white">
+                    <color rgba="1 1 1 1" />
+                </material>
+            </visual>
+        </link>
+        <joint name="base_front_joint" type="fixed">
+            <!-- camera is rotated: it looks to the front and the camera "top"
+                 is on the right wrt/ view (=robot) direction -->
+            <origin xyz="0.1 0 0.3" rpy="0 1.5707963267948966 0"/>
+            <!-- camera is rotated: it looks to the front and the camera "top"
+                 is on the left wrt/ view (=robot) direction
+            <origin xyz="0.1 0 0.3" rpy="0 -1.5707963267948966 3.141592653589793"/>
+            -->
+            <parent link="base_link"/>
+            <child link="web_cam"/>
+        </joint>
+    </xacro:if>
+    <!-- Sonar; all sonars publish in the same frame. -->
+    <link name="sonar">
+        <inertial>
+            <mass value="0.0001"/>
+            <origin xyz="0 0 0"/>
+            <inertia ixx="1" ixy="0" ixz="0" iyy="1" iyz="0" izz="1"/>
+        </inertial>
+        <visual name="pioneer_geom">
+            <origin xyz="0 0 0" rpy="0 0 0"/>
+            <geometry name="pioneer_geom">
+                <mesh filename="package://amr_robots_description/meshes/p3dx_meshes/front_sonar.stl"/>
+            </geometry>
+            <material name="SonarYellow">
+                <color rgba="0.715 0.583 0.210 1.0"/>
+            </material>
+        </visual>
+        <collision>
+            <origin xyz="0 0 0" rpy="0 0 0"/>
+            <geometry>
+                <box size="0 0 0"/>
+            </geometry>
+        </collision>
+    </link>
+    <gazebo reference="sonar">
+        <material value="Gazebo/Yellow"/>
+    </gazebo>
+    <joint name="base_back_joint" type="fixed">
+        <origin xyz="-0.198 0 0.208" rpy="0 0 0"/>
+        <parent link="base_link"/>
+        <child link="sonar"/>
+    </joint>
+    <!-- Caster -->
+    <joint name="base_caster_swivel_joint" type="continuous">
+        <origin xyz="-0.185 0 0.055" rpy="0 0 0"/>
+        <anchor xyz="0 0 0"/>
+        <limit effort="100" velocity="100" k_velocity="0" />
+        <joint_properties damping="0.0" friction="0.0" />
+        <parent link="base_link"/>
+        <child link="caster_swivel"/>
+    </joint>
+    <link name="caster_swivel">
+        <inertial>
+            <mass value="0.1"/>
+            <origin xyz="0 0 0"/>
+            <inertia ixx="0.01" ixy="0" ixz="0"
+                iyy="0.01" iyz="0" izz="0.01"/>
+        </inertial>
+        <visual name="pioneer_geom">
+            <origin xyz="0 0 0" rpy="0 0 0"/>
+            <geometry name="pioneer_geom">
+                <mesh filename="package://amr_robots_description/meshes/p3dx_meshes/caster_swivel.stl"/>
+            </geometry>
+            <material name="caster_swivel">
+                <color rgba="0.5 0.5 0.5 1"/>
+            </material>
+        </visual>
+        <collision>
+            <origin xyz="0 0 0" rpy="0 0 0"/>
+            <geometry>
+                <box size="0 0 0"/>
+            </geometry>
+        </collision>
+    </link>
+    <gazebo reference="caster_swivel">
+        <material value="Gazebo/Grey"/>
+    </gazebo>
+    <!-- Center Wheel + Hubcap -->
+    <link name="caster_hubcap">
+        <inertial>
+            <mass value="0.01"/>
+            <origin xyz="0 0 0"/>
+            <inertia ixx="0.012411765597" ixy="-0.000711733678" ixz="0.00050272983"
+                iyy="0.015218160428" iyz="-0.000004273467" izz="0.011763977943"/>
+        </inertial>
+        <visual name="pioneer_geom">
+            <origin xyz="0 0 0" rpy="0 0 0"/>
+            <geometry name="pioneer_geom">
+                <mesh filename="package://amr_robots_description/meshes/p3dx_meshes/caster_hubcap.stl"/>
+            </geometry>
+            <material name="caster_swivel">
+                <color rgba="0.5 0.5 0.5 1"/>
+            </material>
+        </visual>
+        <collision>
+            <origin xyz="0 0 0" rpy="0 0 0"/>
+            <geometry>
+                <box size="0.05 0.05 0.05"/>
+            </geometry>
+        </collision>
+    </link>
+    <gazebo reference="caster_hubcap">
+        <material value="Gazebo/Grey"/>
+    </gazebo>
+    <joint name="caster_swivel_hubcap_joint" type="continuous">
+        <origin xyz="-0.026 0 -0.016" rpy="0 0 0"/>
+        <axis xyz="0 1 0"/>
+        <anchor xyz="0 0 0"/>
+        <limit effort="100" velocity="100" k_velocity="0" />
+        <joint_properties damping="0.0" friction="0.0" />
+        <parent link="caster_swivel"/>
+        <child link="caster_wheel"/>
+    </joint>
+    <link name="caster_wheel">
+        <inertial>
+            <mass value="0.1"/>
+            <origin xyz="0 0 0"/>
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