Commit message: amigobot: add fov, use more precise urdf model

File: src/amigobot/urdf/amigobot.urdf.xacro (robot description, xacro)
@@ -1,38 +1,102 @@
 <?xml version="1.0"?>
-<!-- created by Jorge Zavala, derived from pioneer3d -->
+<!-- created by Michael Kopp, 2017-02-27, BSD licensed -->
 <robot name="amigobot"
-	xmlns:sensor="http://playerstage.sourceforge.net/gazebo/xmlschema/#sensor"
-	xmlns:controller="http://playerstage.sourceforge.net/gazebo/xmlschema/#controller"
-	xmlns:interface="http://playerstage.sourceforge.net/gazebo/xmlschema/#interface"
-	xmlns:xacro="http://ros.org/wiki/xacro">
-  <!--<include filename="$(find amr_robots_description)/urdf/materials.xacro"/>-->
-  <xacro:include filename="$(find amr_robots_description)/urdf/pioneer3dx_wheel.xacro"/>
-    <!-- Chassis -->
-	<link name="base_link">
-		<inertial>
-			<mass value="3.5"/>
-			<!--<origin xyz="-0.025 0 -0.223"/>-->
-			<origin xyz="0 0 0"/>
-            <!-- inertia: the robot is modeled as filled cylinder with r=0.2m, h=0.2m, m=3.5kg -->
-			<inertia ixx="0.44" ixy="0" ixz="0"
-				 iyy="0.44" iyz="0"
-				 izz="0.07"/>
-		</inertial>
-		<visual>
-			<origin xyz="-0.045 0 0.148" rpy="0 0 0"/>
-			<geometry name="pioneer_geom">
-				<mesh filename="package://amr_robots_description/meshes/p3dx_meshes/chassis.stl"/>
-			</geometry>
-			<material name="ChassisRed">
-				<color rgba="0.851 0.0 0.0 1.0"/>
-			</material>
-		</visual>
-		<collision>
-			<origin xyz="0 0 0" rpy="0 0 0"/>
-				<geometry>
-					<box size="0.01 0.01 0.01"/>
-				</geometry>
-		</collision>
-	</link>
+    xmlns:sensor="http://playerstage.sourceforge.net/gazebo/xmlschema/#sensor"
+    xmlns:controller="http://playerstage.sourceforge.net/gazebo/xmlschema/#controller"
+    xmlns:interface="http://playerstage.sourceforge.net/gazebo/xmlschema/#interface"
+    xmlns:xacro="http://ros.org/wiki/xacro">
+    <!-- chassis -->
+    <link name="base_link">
+        <visual>
+            <origin xyz="0.05 0 0.08" /> <!-- 3cm above floor, height 10cm; center at 8cm -->
+            <geometry>
+                <cylinder length="0.10" radius="0.1" />
+            </geometry>
+            <material name="robot_color"> <color rgba="1 0 0 1" /> </material>
+        </visual>
+        <visual>
+            <origin xyz="-0.06 0 0.08" />
+            <geometry>
+                <cylinder length="0.10" radius="0.1" />
+            </geometry>
+                <material name="green"> <color rgba="0 1 0 0.5" /> </material>
+        </visual>
+        <visual>
+            <origin xyz="-0.02 0 0.08" />
+            <geometry>
+                <box size="0.12 0.28 0.1" />
+            </geometry>
+            <material name="robot_color" />
+        </visual>
+        <visual>
+            <origin xyz="-0.08 0.1 0.08" /> <!-- x is box border -->
+            <geometry>
+                <cylinder length="0.10" radius="0.04" />
+            </geometry>
+            <material name="robot_color" />
+        </visual>
+        <visual>
+            <origin xyz="-0.08 -0.1 0.08" />
+            <geometry>
+                <cylinder length="0.10" radius="0.04" />
+            </geometry>
+            <material name="robot_color" />
+        </visual>
+    </link>
+    <!-- sonar; global frame in which sonar messages are published -->
+    <link name="sonar" />
+    <joint name="sonar_to_base_link" type="fixed">
+        <parent link="base_link" />
+        <child link="sonar" />
+        <origin xyz="0 0 0.11" />
+    </joint>
+    <!-- individual sonars -->
+    <xacro:macro name="single_sonar" params="num x y theta">
+        <link name="sonar_${num}">
+            <visual>
+                <!-- flat cylinder; flat side is in x direction, rotate in joint
+                 appropriately -->
+                <origin xyz="0 0 0" rpy="0 1.5707963267948966 0" />
+                <geometry>
+                    <cylinder length="0.01" radius="0.02" />
+                </geometry>
+                <material name="yellow">
+                    <color rgba="1 1 0 1" />
+                </material>
+            </visual>
+        </link>
+        <joint name="sonar_${num}_to_base_link" type="fixed">
+            <parent link="base_link" />
+            <child link="sonar_${num}" />
+            <origin xyz="${x} ${y} 0.11" rpy="0 0 ${theta}" />
+        </joint>
+    </xacro:macro>
+    <!-- sonar poses in x [mm], y [mm], theta [rad] of robot system
+          at 70, 100, 1.5708
+          at 125, 75, 0.715585
+          at 144, 30, 0.261799
+          at 144, -30, -0.261799
+          at 120, -75, -0.715585
+          at 70, -100, -1.5708
+          at -146, -58, -2.53073
+          at -146, 58, 2.53073
+          -->
+    <xacro:single_sonar num="0" x="0.07" y="0.1" theta="1.5707963267948966" />
+    <xacro:single_sonar num="1" x="0.125" y="0.075" theta="0.715585" />
+    <xacro:single_sonar num="2" x="0.144" y="0.03" theta="0.261799" />
+    <xacro:single_sonar num="3" x="0.144" y="-0.03" theta="-0.261799" />
+    <xacro:single_sonar num="4" x="0.125" y="-0.075" theta="-0.715585" />
+    <xacro:single_sonar num="5" x="0.07" y="-0.1" theta="-1.5707963267948966" />
+    <xacro:single_sonar num="6" x="-0.146" y="-0.058" theta="-2.53073" />
+    <xacro:single_sonar num="7" x="-0.146" y="0.058" theta="2.53073" />
+    <!-- stuff mounted on the robot should refer to this
+         The robot has a small black dot at the "center" of the top_plate frame.
+         -->
+    <link name="top_plate" />
+    <joint name="top_plate_to_base_link" type="fixed">
+        <parent link="base_link" />
+        <child link="top_plate" />
+        <origin xyz="0 0 0.13" />
+    </joint>
     <!-- Camera; mounted on top front of robot; rotated to the right.
          load the xacro with
@@ -45,275 +109,22 @@
     <xacro:if value="$(arg use_web_cam)">
         <link name="web_cam">
-            <inertial>
-                <mass value="0.05" />
-                <origin xyz="0 0 0" rpy="0 0 0"/>
-                <inertia ixx="1e-6" ixy="0" ixz="0" iyy="1e-6" iyz="0" izz="1e-6" />
-            </inertial>
-            <collision>
-                <origin xyz="0 0 0" rpy="0 0 0"/>
-                <geometry>
-                    <box size="0.2 0.12 0.2" /> <!-- larger box to include stand -->
-                </geometry>
-            </collision>
             <visual>
-                <origin xyz="0 0 0" rpy="0 0 0"/>
                 <geometry>
                     <box size="0.07 0.1 0.025"/>
                 </geometry>
-                <material name="white">
-                    <color rgba="1 1 1 1" />
-                </material>
+                <material name="white"> <color rgba="1 1 1 1" /> </material>
             </visual>
         </link>
-        <joint name="base_front_joint" type="fixed">
-            <!-- camera is rotated: it looks to the front and the camera "top"
+        <joint name="camera_to_top_plate" type="fixed">
+            <!-- camera is rotated; it looks to the front and the camera "top"
                  is on the right wrt/ view (=robot) direction -->
-            <origin xyz="0.1 0 0.3" rpy="0 1.5707963267948966 0"/>
-            <!-- camera is rotated: it looks to the front and the camera "top"
+            <origin xyz="0.09 0 0.1" rpy="0 1.5707963267948966 0"/>
+            <!-- camera is rotated; it looks to the front and the camera "top"
                  is on the left wrt/ view (=robot) direction
-            <origin xyz="0.1 0 0.3" rpy="0 -1.5707963267948966 3.141592653589793"/>
+            <origin xyz="0.09 0 0.1" rpy="0 -1.5707963267948966 3.141592653589793"/>
             -->
-            <parent link="base_link"/>
+            <parent link="top_plate"/>
             <child link="web_cam"/>
         </joint>
     </xacro:if>
-    <!-- Sonar; all sonars publish in the same frame. -->
-    <link name="sonar">
-        <inertial>
-            <mass value="0.0001"/>
-            <origin xyz="0 0 0"/>
-            <inertia ixx="1" ixy="0" ixz="0" iyy="1" iyz="0" izz="1"/>
-        </inertial>
-        <visual name="pioneer_geom">
-            <origin xyz="0 0 0" rpy="0 0 0"/>
-            <geometry name="pioneer_geom">
-                <mesh filename="package://amr_robots_description/meshes/p3dx_meshes/front_sonar.stl"/>
-            </geometry>
-            <material name="SonarYellow">
-                <color rgba="0.715 0.583 0.210 1.0"/>
-            </material>
-        </visual>
-        <collision>
-            <origin xyz="0 0 0" rpy="0 0 0"/>
-            <geometry>
-                <box size="0 0 0"/>
-            </geometry>
-        </collision>
-    </link>
-    <gazebo reference="sonar">
-        <material value="Gazebo/Yellow"/>
-    </gazebo>
-    <joint name="base_back_joint" type="fixed">
-        <origin xyz="-0.198 0 0.208" rpy="0 0 0"/>
-        <parent link="base_link"/>
-        <child link="sonar"/>
-    </joint>
-    <!-- Caster -->
-    <joint name="base_caster_swivel_joint" type="continuous">
-        <origin xyz="-0.185 0 0.055" rpy="0 0 0"/>
-        <anchor xyz="0 0 0"/>
-        <limit effort="100" velocity="100" k_velocity="0" />
-        <joint_properties damping="0.0" friction="0.0" />
-        <parent link="base_link"/>
-        <child link="caster_swivel"/>
-    </joint>
-    <link name="caster_swivel">
-        <inertial>
-            <mass value="0.1"/>
-            <origin xyz="0 0 0"/>
-            <inertia ixx="0.01" ixy="0" ixz="0"
-                iyy="0.01" iyz="0" izz="0.01"/>
-        </inertial>
-        <visual name="pioneer_geom">
-            <origin xyz="0 0 0" rpy="0 0 0"/>
-            <geometry name="pioneer_geom">
-                <mesh filename="package://amr_robots_description/meshes/p3dx_meshes/caster_swivel.stl"/>
-            </geometry>
-            <material name="caster_swivel">
-                <color rgba="0.5 0.5 0.5 1"/>
-            </material>
-        </visual>
-        <collision>
-            <origin xyz="0 0 0" rpy="0 0 0"/>
-            <geometry>
-                <box size="0 0 0"/>
-            </geometry>
-        </collision>
-    </link>
-    <gazebo reference="caster_swivel">
-        <material value="Gazebo/Grey"/>
-    </gazebo>
-    <!-- Center Wheel + Hubcap -->
-    <link name="caster_hubcap">
-        <inertial>
-            <mass value="0.01"/>
-            <origin xyz="0 0 0"/>
-            <inertia ixx="0.012411765597" ixy="-0.000711733678" ixz="0.00050272983"
-                iyy="0.015218160428" iyz="-0.000004273467" izz="0.011763977943"/>
-        </inertial>
-        <visual name="pioneer_geom">
-            <origin xyz="0 0 0" rpy="0 0 0"/>
-            <geometry name="pioneer_geom">
-                <mesh filename="package://amr_robots_description/meshes/p3dx_meshes/caster_hubcap.stl"/>
-            </geometry>
-            <material name="caster_swivel">
-                <color rgba="0.5 0.5 0.5 1"/>
-            </material>
-        </visual>
-        <collision>
-            <origin xyz="0 0 0" rpy="0 0 0"/>
-            <geometry>
-                <box size="0.05 0.05 0.05"/>
-            </geometry>
-        </collision>
-    </link>
-    <gazebo reference="caster_hubcap">
-        <material value="Gazebo/Grey"/>
-    </gazebo>
-    <joint name="caster_swivel_hubcap_joint" type="continuous">
-        <origin xyz="-0.026 0 -0.016" rpy="0 0 0"/>
-        <axis xyz="0 1 0"/>
-        <anchor xyz="0 0 0"/>
-        <limit effort="100" velocity="100" k_velocity="0" />
-        <joint_properties damping="0.0" friction="0.0" />
-        <parent link="caster_swivel"/>
-        <child link="caster_wheel"/>
-    </joint>
-    <link name="caster_wheel">
-        <inertial>
-            <mass value="0.1"/>
-            <origin xyz="0 0 0"/>
-            <inertia ixx="0.012411765597" ixy="-0.000711733678" ixz="0.00050272983"
-                iyy="0.015218160428" iyz="-0.000004273467" izz="0.011763977943"/>
-        </inertial>
-        <visual name="pioneer_geom">
-            <origin xyz="0 0 0" rpy="0 0 0"/>
-            <geometry name="pioneer_geom">
-                <mesh filename="package://amr_robots_description/meshes/p3dx_meshes/caster_wheel.stl"/>
-            </geometry>
-            <material name="WheelBlack">
-                <color rgba="0.117 0.117 0.117 1"/>
-            </material>
-        </visual>
-        <collision>
-            <origin xyz="0 0 0" rpy="${-3.1415927/2.0} 0 0"/>
-            <geometry>
-                <!--<mesh filename="package://amr_robots_description/meshes/p3dx_meshes/caster_wheel.stl"/>-->
-                <cylinder radius="0.0375" length="0.01"/>
-            </geometry>
-        </collision>
-    </link>
-    <gazebo reference="left_hub">
-        <material value="Gazebo/Yellow"/>
-    </gazebo>
-    <joint name="caster_wheel_joint" type="fixed">
-        <origin xyz="-0.0035 0 -0.001" rpy="0 0 0"/>
-        <parent link="caster_wheel"/>
-        <child link="caster_hubcap"/>
-    </joint>
-    <link name="left_hub">
-        <visual>
-            <origin xyz="0 0 0" rpy="0 0 0"/>
-            <geometry>
-                <mesh filename="package://amr_robots_description/meshes/p3dx_meshes/left_hubcap.stl"/>
-            </geometry>
-            <material name="HubcapYellow">
-                <color rgba="1.0 0.811 0.151 1.0"/>
-            </material>
-        </visual>
-        <collision>
-            <origin xyz="0 0 0" rpy="${-3.1415927/2.0} 0 0"/>
-            <geometry>
-                <!--<mesh filename="package://amr_robots_description/meshes/p3dx_meshes/caster_wheel.stl"/>-->
-                <cylinder radius="0.09" length="0.01"/>
-            </geometry>
-        </collision>
-    </link>
-    <joint name="left_hub_joint" type="fixed">
-        <origin xyz="0 0.15 0.08" rpy="0 0 0"/>
-        <parent link="base_link"/>
-        <child link="left_hub"/>
-        <axis xyz="0 1 0"/>
-    </joint>
-    <link name="left_wheel">
-        <visual>
-            <origin xyz="0 0 0" rpy="0 0 0"/>
-            <geometry>
-                <mesh filename="package://amr_robots_description/meshes/p3dx_meshes/left_wheel.stl"/>
-            </geometry>
-            <material name="WheelBlack">
-                <color rgba="0.117 0.117 0.117 1"/>
-            </material>
-        </visual>
-    </link>
-    <joint name="left_wheel_joint" type="fixed"> <!-- type="continuous" -->
-        <origin xyz="0 0 0" rpy="0 0 0"/>
-        <parent link="left_hub"/>
-        <child link="left_wheel"/>
-    </joint>
-    <gazebo reference="left_wheel_joint">
-        <material value="Gazebo/Black"/>
-    </gazebo>
-    <link name="right_hub">
-        <visual>
-            <origin xyz="0 0 0" rpy="0 0 0"/>
-            <geometry>
-                <mesh filename="package://amr_robots_description/meshes/p3dx_meshes/right_hubcap.stl"/>
-            </geometry>
-            <material name="HubcapYellow">
-                <color rgba="1.0 0.811 0.151 1.0"/>
-            </material>
-        </visual>
-        <collision>
-            <origin xyz="0 0 0" rpy="${-3.1415927/2.0} 0 0"/>
-            <geometry>
-                <!--<mesh filename="package://amr_robots_description/meshes/p3dx_meshes/caster_wheel.stl"/>-->
-                <cylinder radius="0.09" length="0.01"/>
-            </geometry>
-        </collision>
-    </link>
-    <gazebo reference="right_hub">
-        <material value="Gazebo/Yellow"/>
-    </gazebo>
-    <joint name="right_hub_joint" type="fixed">
-        <origin xyz="0 -0.15 0.08" rpy="0 0 0"/>
-        <parent link="base_link"/>
-        <child link="right_hub"/>
-        <axis xyz="0 1 0"/>
-    </joint>
-    <link name="right_wheel">
-        <visual>
-            <origin xyz="0 0 0" rpy="0 0 0"/>
-            <geometry>
-                <mesh filename="package://amr_robots_description/meshes/p3dx_meshes/right_wheel.stl"/>
-            </geometry>
-            <material name="WheelBlack">
-                <color rgba="0.117 0.117 0.117 1"/>
-            </material>
-        </visual>
-    </link>
-    <joint name="right_wheel_joint" type="fixed"> <!-- type="continuous" -->
-        <origin xyz="0 0 0" rpy="0 0 0"/>
-        <parent link="right_hub"/>
-        <child link="right_wheel"/>
-    </joint>
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
Commit message: amigobot: use better camera position (no stand); add to urdf

File: src/amigobot/urdf/amigobot.urdf.xacro (robot description, xacro)
@@ -99,17 +99,42 @@
         <origin xyz="0 0 0.13" />
     </joint>
-    <!-- Camera; mounted on top front of robot; rotated to the right.
+    <!-- Camera; mounted on top front of robot
          load the xacro with
-         <param name="robot_description" command="$(find xacro)/xacro.py $(arg model) use_web_cam:=false" />
+         <param name="robot_description" command="$(find xacro)/xacro $(arg model) web_cam_position:='false'" />
          to not add a camera.
          For a camera, the z axis is in the direction of the view, x goes to
          the right (wrt/ view direction) and y downwards.
+         Parameters to place the web cam:
+         web_cam_position can be a triple x y z; relative position from the top
+            plate origin (small black plastic disc)
+            defaults to "0.063 0 0.054" which is the value for the lens of an
+            edimax_ic_3115w camera mounted directly on the robot (i.e. no
+            stand) s.th. the indentation that runs around the camera directly
+            touches the second screw holes from the front of the robot.
+            If this is 'false', no web cam is included in the urdf.
+         web_cam_rotation can be a triple roll pitch yaw for the camera
+            rotation.
+            The default is "pi/2 pi pi/2 " which is a camera that looks to the
+            front of the robot (i.e. z_camera is x_robot, y_camera is -z_robot).
+            Note: You can use this applett
+            http://www.ctralie.com/Teaching/COMPSCI290/Materials/EulerAnglesViz/
+            to easily determine rpy values.
+            Example values:
+            - "0 1.5707963267948966 0": camera looks to the front direction of
+                the robot and the camera "top" is on the right wrt/ view
+                (=robot) direction.
+            - "0 -1.5707963267948966 3.141592653589793": like above but camera
+                "top" is on the left wrt/ view direction.
          -->
-    <xacro:arg name="use_web_cam" default="true"/>
-    <xacro:if value="$(arg use_web_cam)">
+    <!-- arguments to this xacro file -->
+    <xacro:arg name="web_cam_position" default="0.063 0 0.054" />
+    <xacro:arg name="web_cam_rotation" default="1.5707963267948966 3.141592653589793 1.5707963267948966" />
+    <!-- make them parameter in xacro -->
+    <xacro:property name="web_cam_position_prop" value="$(arg web_cam_position)"/>
+    <xacro:if value="${web_cam_position_prop != 'false'}">
         <link name="web_cam">
             <visual>
                 <geometry>
-                    <box size="0.07 0.1 0.025"/>
+                    <box size="0.07 0.1 0.025"/> <!-- size of an edimax_ic_3115w -->
                 </geometry>
                 <material name="white"> <color rgba="1 1 1 1" /> </material>
@@ -117,11 +142,5 @@
         </link>
         <joint name="camera_to_top_plate" type="fixed">
-            <!-- camera is rotated; it looks to the front and the camera "top"
-                 is on the right wrt/ view (=robot) direction -->
-            <origin xyz="0.09 0 0.1" rpy="0 1.5707963267948966 0"/>
-            <!-- camera is rotated; it looks to the front and the camera "top"
-                 is on the left wrt/ view (=robot) direction
-            <origin xyz="0.09 0 0.1" rpy="0 -1.5707963267948966 3.141592653589793"/>
-            -->
+            <origin xyz="$(arg web_cam_position)" rpy="$(arg web_cam_rotation)"/>
             <parent link="top_plate"/>
             <child link="web_cam"/>
